Commit message: Added inertial properties to the bot and correctly wrote the launch file which now open both gazebo and rviz

File: urdf/robot.urdf.xacro (robot description, xacro)
@@ -11,4 +11,21 @@
             </geometry>
         </visual>
+        <inertial>
+            <mass value="1.0"/>
+            <origin xyz="0.0 0.0 0.0" rpy="0.0 0.0 0.0" />
+            <inertia ixx="0.01" ixy="0.0" ixz="0.0" iyy="0.01" iyz="0.0" izz="0.01"/>
+        </inertial>
+        <collision>
+            <origin xyz="0.0 0.0 0.0" rpy="0.0 0.0 0.0" />
+            <geometry>
+                <box size="0.15 0.15 0.05"/>
+            </geometry>
+        </collision>
+        <gazebo reference="chassis">
+            <material>Gazebo/Grey</material>
+            <selfCollide>true</selfCollide>
+            <mu1>0.5</mu1>
+            <mu2>0.5</mu2>
+        </gazebo>
     </link>
     <link name="right_wheel">
@@ -17,13 +34,30 @@
                 <cylinder radius="0.03" length="0.02"/>
             </geometry>
-                <origin xyz="0 -0.085 0" rpy=" 1.57 0.0 0.0" />
-                <material name="black">
-                    <color rgba="0 0 0 1"/>
-                </material>
+            <origin xyz="0 0 0" rpy="1.57 0.0 0.0" />
+            <material name="black">
+                <color rgba="0 0 0 1"/>
+            </material>
         </visual>
+        <collision>
+            <geometry>
+                <cylinder radius="0.03" length="0.02"/>
+            </geometry>
+            <origin xyz="0 0 0" rpy="1.57 0.0 0.0" />
+        </collision>
+        <inertial>
+            <mass value="0.05"/>
+            <origin xyz="0 0 0" rpy="0 0 0"/>
+            <inertia ixx="0.0001" ixy="0.0" ixz="0.0" iyy="0.0001" iyz="0.0" izz="0.0001"/>
+        </inertial>
+        <gazebo reference="right_wheel">
+            <material>Gazebo/Black</material>
+            <selfCollide>true</selfCollide>
+            <mu1>1.0</mu1>
+            <mu2>1.0</mu2>
+        </gazebo>
     </link>
     <link name="left_wheel">
         <visual>
-            <origin xyz="0 0.085 0" rpy=" 1.57 0.0 0.0" />
+            <origin xyz="0 0 0" rpy=" 1.57 0.0 0.0" />
             <geometry>
                 <cylinder radius="0.03" length="0.02"/>
@@ -33,4 +67,21 @@
                 </material>
         </visual>
+               <collision>
+            <geometry>
+                <cylinder radius="0.03" length="0.02"/>
+            </geometry>
+            <origin xyz="0 0 0" rpy="1.57 0.0 0.0" />
+        </collision>
+        <inertial>
+            <mass value="0.05"/>
+            <origin xyz="0 0 0" rpy="0 0 0"/>
+            <inertia ixx="0.0001" ixy="0.0" ixz="0.0" iyy="0.0001" iyz="0.0" izz="0.0001"/>
+        </inertial>
+        <gazebo reference="left_wheel">
+            <material>Gazebo/Black</material>
+            <selfCollide>true</selfCollide>
+            <mu1>1.0</mu1>
+            <mu2>1.0</mu2>
+        </gazebo>
     </link>
     <link name="castor_wheel">
@@ -44,7 +95,18 @@
                 </material>
         </visual>
+        <collision>
+            <geometry>
+                <sphere radius="0.01"/>
+                <origin xyz="0.0 0.0 0.0" />
+            </geometry>
+        </collision>
+        <inertial>
+            <mass value="0.01"/>
+            <origin xyz="0 0 0" rpy="0 0 0"/>
+            <inertia ixx="0.00001" ixy="0.0" ixz="0.0" iyy="0.00001" iyz="0.0" izz="0.00001"/>
+        </inertial>
     </link>
     <xacro:property name="sensor_x" value="0.040"/>
-    <xacro:macro name="ir_sensors" params="name y">
+    <xacro:macro name="ir_sensors" params="name y">  <!-- Keep this line -->
         <link name="${name}">
             <visual>
@@ -73,5 +135,5 @@
         <parent link="chassis"/>
         <child link="left_wheel"/>
-        <origin xyz="-0.05 0 -0.01" />
+        <origin xyz="-0.05 0.085 -0.01" />
         <axis xyz="0 1 0"/>
     </joint>
@@ -79,5 +141,5 @@
         <parent link="chassis"/>
         <child link="right_wheel"/>
-        <origin xyz="-0.05 0 -0.01" />
+        <origin xyz="-0.05 -0.085 -0.01" />
         <axis xyz="0 1 0"/>
     </joint>

Commit message: moved from 5 ir sensors to camera module

File: urdf/robot.urdf.xacro (robot description, xacro)
@@ -12,5 +12,5 @@
         </visual>
         <inertial>
-            <mass value="1.0"/>
+            <mass value="3.0"/>
             <origin xyz="0.0 0.0 0.0" rpy="0.0 0.0 0.0" />
             <inertia ixx="0.01" ixy="0.0" ixz="0.0" iyy="0.01" iyz="0.0" izz="0.01"/>
@@ -46,5 +46,5 @@
         </collision>
         <inertial>
-            <mass value="0.05"/>
+            <mass value="0.1"/>
             <origin xyz="0 0 0" rpy="0 0 0"/>
             <inertia ixx="0.0001" ixy="0.0" ixz="0.0" iyy="0.0001" iyz="0.0" izz="0.0001"/>
@@ -74,5 +74,5 @@
         </collision>
         <inertial>
-            <mass value="0.05"/>
+            <mass value="0.1"/>
             <origin xyz="0 0 0" rpy="0 0 0"/>
             <inertia ixx="0.0001" ixy="0.0" ixz="0.0" iyy="0.0001" iyz="0.0" izz="0.0001"/>
@@ -106,34 +106,60 @@
             <inertia ixx="0.00001" ixy="0.0" ixz="0.0" iyy="0.00001" iyz="0.0" izz="0.00001"/>
         </inertial>
+        <gazebo reference="castor_wheel">
+            <material>Gazebo/Red</material>
+            <mu1>0.001</mu1>  <!-- Static friction -->
+            <mu2>0.001</mu2>  <!-- Dynamic friction -->
+            <kp>1000000.0</kp>  <!-- Contact stiffness -->
+            <kd>100.0</kd>     <!-- Contact damping -->
+        </gazebo>
     </link>
-    <xacro:property name="sensor_x" value="0.040"/>
-    <xacro:macro name="ir_sensors" params="name y">  <!-- Keep this line -->
-        <link name="${name}">
-            <visual>
-                <origin xyz="${sensor_x} ${y} -0.01" />
-                <geometry>
-                    <box size="0.01 0.01 0.01"/>
-                </geometry>
-                <material name="pink">
-                    <color rgba="1 0.5 0.5 1"/>
-                </material>
-            </visual>
-        </link>
-        <joint name="${name}_joint" type="fixed">
-            <parent link="chassis"/>
-            <child link="${name}"/>
-            <origin xyz="${sensor_x} ${y} -0.01" />
-        </joint>
-    </xacro:macro>
-    <xacro:ir_sensors name="ir_lout"  y="0.035" />
-    <xacro:ir_sensors name="ir_rout" y="-0.035" />
-    <xacro:ir_sensors name="ir_rin"  y="-0.0175" />
-    <xacro:ir_sensors name="ir_lin"  y="0.0175" />
-    <xacro:ir_sensors name="ir_centre" y="0" />
+    <link name="camera_link">
+      <visual>
+        <origin xyz="0 0 0"/>
+        <geometry>
+          <box size="0.05 0.04 0.01"/>
+        </geometry>
+        <material name="black">
+          <color rgba="0 0 0 1"/>
+        </material>
+      </visual>
+    </link>
+    <joint name="camera_joint" type="fixed">
+      <parent link="chassis"/>
+      <child link="camera_link"/>
+      <origin xyz="0.075 0 0.03" rpy="0 0 0" />
+    </joint>
+    <gazebo reference="camera_link">
+      <sensor type="camera" name="line_follower_camera">
+        <always_on>true</always_on>
+        <update_rate>30</update_rate>
+        <camera>
+          <horizontal_fov>1.0</horizontal_fov>
+          <image>
+            <width>320</width>
+            <height>240</height>
+            <format>R8G8B8</format>
+          </image>
+          <clip>
+            <near>0.01</near>
+            <far>10</far>
+          </clip>
+        </camera>
+        <plugin name="gazebo_ros_camera" filename="libgazebo_ros_camera.so">
+          <ros>
+            <namespace>/camera</namespace>
+          </ros>
+          <camera_name>line_follower</camera_name>
+          <image_topic_name>image_raw</image_topic_name>
+          <camera_info_topic_name>camera_info</camera_info_topic_name>
+          <frame_name>camera_link</frame_name>
+        </plugin>
+      </sensor>
+    </gazebo>
     <!-- joint ahead -->
     <joint name="left_wheel_joint" type="continuous">
         <parent link="chassis"/>
         <child link="left_wheel"/>
-        <origin xyz="-0.05 0.085 -0.01" />
+        <origin xyz="-0.055 0.085 -0.005" />
         <axis xyz="0 1 0"/>
     </joint>
@@ -141,11 +167,12 @@
         <parent link="chassis"/>
         <child link="right_wheel"/>
-        <origin xyz="-0.05 -0.085 -0.01" />
+        <origin xyz="-0.055 -0.085 -0.005" />
         <axis xyz="0 1 0"/>
     </joint>
-    <joint name="castor_wheel_joint" type="fixed">
+    <joint name="castor_wheel_joint" type="continuous">
         <parent link="chassis"/>
         <child link="castor_wheel"/>
         <origin xyz="0.050 0 -0.025" />
+        <axis xyz="0 1 0"/>
     </joint>
     <!-- ROBOT MOVEMENT STUFF AHEAD  -->

Commit message: made the code a little clean

File: urdf/robot.urdf.xacro (robot description, xacro)
@@ -1,4 +1,5 @@
 <?xml version="1.0"?>
 <robot name="line_maze_solver" xmlns:xacro="http://www.ros.org/wiki/xacro">
+    <xacro:include filename="camera.xacro"/>
     <link name="chassis">
         <visual>
@@ -114,47 +115,4 @@
         </gazebo>
     </link>
-    <link name="camera_link">
-      <visual>
-        <origin xyz="0 0 0"/>
-        <geometry>
-          <box size="0.05 0.04 0.01"/>
-        </geometry>
-        <material name="black">
-          <color rgba="0 0 0 1"/>
-        </material>
-      </visual>
-    </link>
-    <joint name="camera_joint" type="fixed">
-      <parent link="chassis"/>
-      <child link="camera_link"/>
-      <origin xyz="0.075 0 0.03" rpy="0 0 0" />
-    </joint>
-    <gazebo reference="camera_link">
-      <sensor type="camera" name="line_follower_camera">
-        <always_on>true</always_on>
-        <update_rate>30</update_rate>
-        <camera>
-          <horizontal_fov>1.0</horizontal_fov>
-          <image>
-            <width>320</width>
-            <height>240</height>
-            <format>R8G8B8</format>
-          </image>
-          <clip>
-            <near>0.01</near>
-            <far>10</far>
-          </clip>
-        </camera>
-        <plugin name="gazebo_ros_camera" filename="libgazebo_ros_camera.so">
-          <ros>
-            <namespace>/camera</namespace>
-          </ros>
-          <camera_name>line_follower</camera_name>
-          <image_topic_name>image_raw</image_topic_name>
-          <camera_info_topic_name>camera_info</camera_info_topic_name>
-          <frame_name>camera_link</frame_name>
-        </plugin>
-      </sensor>
-    </gazebo>
     <!-- joint ahead -->
     <joint name="left_wheel_joint" type="continuous">
