Commit message: bot and algorithm bot are working just need bit of fine tunings

File: urdf/camera.xacro (robot description, xacro)
@@ -10,5 +10,5 @@
             <origin xyz="0 0 0"/>
             <geometry>
-              <box size="0.05 0.04 0.01"/>
+              <box size="0.02 0.04 0.02"/>
         </geometry>
             <material name="black">

File: urdf/robot.urdf.xacro (robot description, xacro)
@@ -26,6 +26,4 @@
             <material>Gazebo/Grey</material>
             <selfCollide>true</selfCollide>
-            <mu1>0.5</mu1>
-            <mu2>0.5</mu2>
         </gazebo>
     </link>
@@ -47,5 +45,5 @@
         </collision>
         <inertial>
-            <mass value="0.1"/>
+            <mass value="0.001"/>
             <origin xyz="0 0 0" rpy="0 0 0"/>
             <inertia ixx="0.0001" ixy="0.0" ixz="0.0" iyy="0.0001" iyz="0.0" izz="0.0001"/>
@@ -75,5 +73,5 @@
         </collision>
         <inertial>
-            <mass value="0.1"/>
+            <mass value="0.001"/>
             <origin xyz="0 0 0" rpy="0 0 0"/>
             <inertia ixx="0.0001" ixy="0.0" ixz="0.0" iyy="0.0001" iyz="0.0" izz="0.0001"/>

Commit message: optimized the algorithm

File: urdf/camera.xacro (robot description, xacro)
@@ -4,5 +4,5 @@
         <parent link="chassis"/>
         <child link="camera_link"/>
-        <origin xyz="0.075 0 0.03" rpy="0 0 0" />
+        <origin xyz="0.075 0 0.06" rpy="0 0.3 0" />
     </joint>
     <link name="camera_link">
@@ -21,9 +21,14 @@
             <camera>
                 <image>
-                    <width>640</width>
-                    <height>480</height>
+                    <horizontal_fov>2.047</horizontal_fov>
+                    <clip>5</clip>
+                    <update_rate>30</update_rate>
+                    <vertical_fov>0.785</vertical_fov>
+                    <width>800</width>
+                    <height>600</height>
                     <format>R8G8B8</format>
                 </image>
             </camera>
+            <visualize>true</visualize>
             <plugin name="camera_controller" filename="libgazebo_ros_camera.so">
                 <frame_name>camera_link</frame_name>

File: urdf/robot.urdf.xacro (robot description, xacro)
@@ -45,5 +45,5 @@
         </collision>
         <inertial>
-            <mass value="0.001"/>
+            <mass value="1"/>
             <origin xyz="0 0 0" rpy="0 0 0"/>
             <inertia ixx="0.0001" ixy="0.0" ixz="0.0" iyy="0.0001" iyz="0.0" izz="0.0001"/>
@@ -73,5 +73,5 @@
         </collision>
         <inertial>
-            <mass value="0.001"/>
+            <mass value="1"/>
             <origin xyz="0 0 0" rpy="0 0 0"/>
             <inertia ixx="0.0001" ixy="0.0" ixz="0.0" iyy="0.0001" iyz="0.0" izz="0.0001"/>
@@ -107,8 +107,29 @@
         <gazebo reference="castor_wheel">
             <material>Gazebo/Red</material>
-            <mu1>0.001</mu1>  <!-- Static friction -->
-            <mu2>0.001</mu2>  <!-- Dynamic friction -->
-            <kp>1000000.0</kp>  <!-- Contact stiffness -->
-            <kd>100.0</kd>     <!-- Contact damping -->
+        </gazebo>
+    </link>
+    <link name="castor_wheel_lateral">
+        <visual>
+            <origin xyz="0 0 0" />
+                <geometry>
+                    <sphere radius="0.01"/>
+                </geometry>
+                <material name="red">
+                    <color rgba="1 0 0 1"/>
+                </material>
+        </visual>
+        <collision>
+            <geometry>
+                <sphere radius="0.01"/>
+                <origin xyz="0.0 0.0 0.0" />
+            </geometry>
+        </collision>
+        <inertial>
+            <mass value="0.01"/>
+            <origin xyz="0 0 0" rpy="0 0 0"/>
+            <inertia ixx="0.00001" ixy="0.0" ixz="0.0" iyy="0.00001" iyz="0.0" izz="0.00001"/>
+        </inertial>
+        <gazebo reference="castor_wheel">
+            <material>Gazebo/Red</material>
         </gazebo>
     </link>
@@ -128,7 +149,13 @@
     <joint name="castor_wheel_joint" type="continuous">
         <parent link="chassis"/>
+        <child link="castor_wheel_lateral"/>
+        <origin xyz="0.050 0 -0.025" />
+        <axis xyz="0 1 0"/>
+    </joint>
+    <joint name="castor_wheel_joint_lateral" type="continuous">
+        <parent link="chassis"/>
         <child link="castor_wheel"/>
         <origin xyz="0.050 0 -0.025" />
-        <axis xyz="0 1 0"/>
+        <axis xyz="1 0 0"/>
     </joint>
     <!-- ROBOT MOVEMENT STUFF AHEAD  -->
